Commit message: IMU Implimentation with test readings

File: description/mounting_system.xacro (robot description, xacro)
@@ -1,28 +1,9 @@
 <?xml version="1.0"?>
 <robot xmlns:xacro="http://www.ros.org/wiki/xacro">
-     <material name="white">
-        <color rgba="1 1 1 1" />
-    </material>
-    <material name="orange">
-        <color rgba="1 0.3 0.1 1"/>
-    </material>
-    <material name="red">
-        <color rgba="1 0 0 1"/>
-    </material>
-    <material name="blue">
-        <color rgba="0.2 0.2 1 1"/>
-    </material>
-    <material name="black">
-        <color rgba="0 0 0 1"/>
-    </material>
-    <link name="base_link">
-    </link>
     <!-- Stepper Motor Link and Joint-->
-    <joint name="stepper_motor_joint" type="revolute">
-        <parent link="base_link"/>
+    <joint name="stepper_motor_joint" type="fixed">
+        <parent link="imu_angle_adjustment"/>
         <child link="stepper_motor"/>
         <origin xyz="0 0 0" rpy="${pi/2} 0 0"/>
-        <axis xyz="1 1 1"/>
-        <limit effort="1000" lower="-${pi/2}" upper="${pi/2}" velocity="0.5"/>
     </joint>
     <link name="stepper_motor">
@@ -84,46 +65,3 @@
         </collision>
     </link>
-    <!-- LiDAR Link and Joint -->
-    <joint name="lidar_joint" type="fixed">
-        <parent link="mounting_plate_base"/>
-        <child link="lidar_sensor"/>
-        <origin xyz="0 0 0.045" rpy="0 0 ${pi}"/>
-    </joint>
-    <link name="lidar_sensor">
-        <visual>
-            <origin xyz="0 0 -0.00125"/>
-            <geometry>
-                <cylinder radius="0.035" length="0.0225"/>
-                <!-- <mesh filename="file://$(find lidar_converter)/description/RPLiDAR.stl" scale="1 1 1"/> -->
-            </geometry>
-            <material name="black"/>
-        </visual>
-        <collision>
-            <origin xyz="0 0 -0.00125"/>
-            <geometry>
-                <cylinder radius="0.035" length="0.0225"/>
-            </geometry>
-        </collision>
-    </link>
-    <!-- IMU Link and Joint-->
-    <joint name="imu_joint" type="fixed">
-        <parent link="mounting_plate_base"/>
-        <child link="imu_sensor"/>
-        <origin xyz="0 0 0.02"/>
-    </joint>
-    <link name="imu_sensor">
-        <visual>
-            <origin xyz="0 0 0"/>
-            <geometry>
-                <box size="0.02 0.015 0.005"/>
-            </geometry>
-            <material name="red"/>
-        </visual>
-        <collision>
-            <origin xyz="0 0 0"/>
-            <geometry>
-                <box size="0.02 0.015 0.005"/>
-            </geometry>
-        </collision>
-    </link>
 </robot>

File: description/robot_urdf.xacro (robot description, xacro)
@@ -1,4 +1,13 @@
 <?xml version="1.0"?>
 <robot xmlns:xacro="http://www.ros.org/wiki/xacro" name="lidar_assembly">
-    <xacro:include filename="robot_core.xacro" />
+    <!-- Import Colours -->
+    <xacro:include filename="colours.xacro" />
+    <!-- Define Base Link-->
+    <link name="base_link">
+    </link>
+    <!-- <xacro:include filename="imu_standalone.xacro" /> -->
+    <!-- <xacro:include filename="lidar_standalone.xacro" /> -->
+    <xacro:include filename="mounting_system.xacro" />
+    <xacro:include filename="imu.xacro" />
+    <xacro:include filename="lidar.xacro" />
 </robot>
