Commit message: Cleaned, Updated Scan Functionality

File: description/imu.xacro (robot description, xacro)
@@ -5,5 +5,5 @@
         <parent link="mounting_plate_base"/>
         <child link="imu_sensor"/>
-        <origin xyz="0 0 0.02"/>
+        <origin xyz="0 0 0.02" rpy="0 0 0"/>
     </joint>
     <link name="imu_sensor">
@@ -11,5 +11,5 @@
             <origin xyz="0 0 0"/>
             <geometry>
-                <box size="0.02 0.015 0.005"/>
+                <box size="0.025 0.02 0.005"/>
             </geometry>
             <material name="red"/>
@@ -18,5 +18,5 @@
             <origin xyz="0 0 0"/>
             <geometry>
-                <box size="0.02 0.015 0.005"/>
+                <box size="0.025 0.02 0.005"/>
             </geometry>
         </collision>
@@ -26,5 +26,6 @@
         <parent link="base_link"/>
         <child link="imu_angle_adjustment"/>
-        <origin xyz="0 0 0"/>
+        <origin xyz="0 0 0" rpy="0 0 0"/> <!-- ${-1} -->
+        <!--<axis xyz="0 1 0"/>-->
     </joint>
     <link name="imu_angle_adjustment">

Commit message: Updated Model, tweaked point cloud pub & cmake

File: description/imu.xacro (robot description, xacro)
@@ -5,11 +5,11 @@
         <parent link="mounting_plate_base"/>
         <child link="imu_sensor"/>
-        <origin xyz="0 0 0.02" rpy="0 0 0"/>
+        <origin xyz="0 0 0" rpy="0 0 0"/>
     </joint>
     <link name="imu_sensor">
         <visual>
-            <origin xyz="0 0 0"/>
+            <origin xyz="0 0 0.002"/>
             <geometry>
-                <box size="0.025 0.02 0.005"/>
+                <box size="0.025 0.02 0.004"/>
             </geometry>
             <material name="red"/>
@@ -18,5 +18,5 @@
             <origin xyz="0 0 0"/>
             <geometry>
-                <box size="0.025 0.02 0.005"/>
+                <box size="0.025 0.02 0.004"/>
             </geometry>
         </collision>

File: description/lidar.xacro (robot description, xacro)
@@ -5,11 +5,11 @@
         <parent link="mounting_plate_base"/>
         <child link="lidar_sensor"/>
-        <origin xyz="0 0 0.045" rpy="0 0 ${pi}"/>
+        <origin xyz="0 0 0.0466" rpy="0 0 ${pi}"/> <!-- Or 51.6mm depending on top vs base-->
     </joint>
     <link name="lidar_sensor">
         <visual>
-            <origin xyz="0 0 -0.00125"/>
+            <origin xyz="0 0 0"/>
             <geometry>
-                <cylinder radius="0.035" length="0.0225"/>
+                <cylinder radius="0.035" length="0.018"/>
                 <!-- <mesh filename="file://$(find lidar_converter)/description/RPLiDAR.stl" scale="1 1 1"/> -->
             </geometry>
@@ -17,7 +17,7 @@
         </visual>
         <collision>
-            <origin xyz="0 0 -0.00125"/>
+            <origin xyz="0 0 -0.009"/>
             <geometry>
-                <cylinder radius="0.035" length="0.0225"/>
+                <cylinder radius="0.035" length="0.018"/>
             </geometry>
         </collision>

File: description/mounting_system.xacro (robot description, xacro)
@@ -32,14 +32,14 @@
     <link name="mounting_plate_arm">
         <visual>
-            <origin xyz="0 -0.002 -0.0075"/>
+            <origin xyz="0 -0.004 -0.003"/>
             <geometry>
-                <box size="0.025 0.004 0.035"/>
+                <box size="0.040 0.008 0.030"/>
             </geometry>
-            <material name="red"/>
+            <material name="white"/>
         </visual>
         <collision>
-            <origin xyz="0 -0.002 -0.0075"/>
+            <origin xyz="0 -0.004 -0.003"/>
             <geometry>
-                <box size="0.025 0.004 0.035"/>
+                <box size="0.040 0.008 0.030"/>
             </geometry>
         </collision>
@@ -48,18 +48,18 @@
         <parent link="mounting_plate_arm"/>
         <child link="mounting_plate_base"/>
-        <origin xyz="0 -0.039 -0.021"/>
+        <origin xyz="0 -0.0455 -0.013"/>
     </joint>
     <link name="mounting_plate_base">
         <visual>
-            <origin xyz="0 0 -0.002"/>
+            <origin xyz="0 0 -0.0025"/>
             <geometry>
-                <box size="0.09 0.07 0.004"/>
+                <box size="0.09 0.075 0.005"/>
             </geometry>
-            <material name="red"/>
+            <material name="white"/>
         </visual>
         <collision>
             <origin xyz="0 0 -0.002"/>
             <geometry>
-                <box size="0.09 0.07 0.004"/>
+                <box size="0.09 0.075 0.005"/>
             </geometry>
         </collision>
